Commit message: Add CAD models and target markers for inverse kinematics testing
- Added QarmBase.stl and QarmHoop.stl mesh files for platform and hoop visualization
- Updated QARM.urdf to reference new mesh files
- Enhanced sim/env.py with comprehensive simulation features:
  * Added base fixture (platform) loading with QarmBase.stl mesh
  * Added DarmHoop loading with QarmHoop.stl mesh (with fallback torus representation)
  * Implemented target coordinate markers for inverse kinematics testing:
    - Three target markers with different colors (red, blue, orange)
    - Floating coordinate text labels above each marker
    - Configurable target positions for student testing
  * Positioned hoop 30cm forward on platform to avoid Q arm base occlusion
  * Added proper coordinate recording and logging

Target coordinates:
- Target 1 (Red): (0.10, 0.20, 0.12)
- Target 2 (Blue): (0.25, 0.30, 0.40)
- Target 3 (Orange): (0.15, 0.40, 0.06)

This update enables students to test their inverse kinematics algorithms
by attempting to reach the three target coordinates in the simulation.

File: qarm/urdf/QARM.urdf (robot description, URDF)
Before this commit: robot QARM, 6 links, 5 joints
Links:
- link BICEP: geometry collision mesh filename=../meshes/BICEP.STL; visual mesh filename=../meshes/BICEP.STL
- link END-EFFECTOR: geometry collision mesh filename=../meshes/END-EFFECTOR.STL; visual mesh filename=../meshes/END-EFFECTOR.STL
- link FOREARM: geometry collision mesh filename=../meshes/FOREARM.STL; visual mesh filename=../meshes/FOREARM.STL
- link YAW: geometry collision mesh filename=../meshes/YAW.STL; visual mesh filename=../meshes/YAW.STL
- link base_link: geometry collision mesh filename=../meshes/base_link.STL; visual mesh filename=../meshes/base_link.STL

Commit message: - stripped down the simulation - focused on a fixed gripper system

File: qarm/urdf/QARM.urdf (robot description, URDF)
Before this commit: robot QARM, 6 links, 5 joints
Links:
- link END-EFFECTOR: geometry collision mesh filename=package://QARM/meshes/END-EFFECTOR.STL; collision mesh filename=package://QARM/meshes/Gripper.stl
