Commit message: Add gripper base + link1a and make Panda viewer load URDF visuals
- extend QARM URDF with GRIPPER_BASE (fixed to END-EFFECTOR) and GRIPPER_LINK1A meshes; drop legacy Gripper.stl visual
- scale gripper meshes to meters and (current state) leave link1a joint at origin with +X axis and wide limits
- rework Panda viewer to build visuals from Bullet URDF data (path/offset/scale/orientation) with fallbacks, and add optional mesh reload flag
- add --reload-meshes CLI flag and RELOAD_MESHES toggle in student scripts; fix Panda import block syntax

File: sim/qarm/urdf/QARM.urdf (robot description, URDF)
Before this commit: robot QARM, 6 links, 5 joints
Links:
- added link GRIPPER_BASE, mass 0.05; collision mesh filename=package://QARM/meshes/gripper-base.stl scale=0.001 0.001 0.001; visual mesh filename=package://QARM/meshes/gripper-base.stl scale=0.001 0.001 0.001
- added link GRIPPER_LINK1A, mass 0.02; collision mesh filename=package://QARM/meshes/gripper-link1a.stl scale=0.001 0.001 0.001; visual mesh filename=package://QARM/meshes/gripper-link1a.stl scale=0.001 0.001 0.001
- link END-EFFECTOR: geometry collision mesh filename=package://QARM/meshes/END-EFFECTOR.STL; visual mesh filename=package://QARM/meshes/END-EFFECTOR.STL
Joints:
- added joint GRIPPER_BASE_FIXED: type fixed, parent END-EFFECTOR, child GRIPPER_BASE, origin xyz=0 0 0 rpy=0 0 0
- added joint GRIPPER_JOINT1A: type revolute, parent GRIPPER_BASE, child GRIPPER_LINK1A, origin xyz=0.02 -0.0303 0.0406 rpy=0 0 0, axis 1 0 0, limit lower=-3.14159 upper=3.14159 effort=0 velocity=0

Commit message: Add remaining gripper links and viewer mappings - add GRIPPER_LINK1B plus cloned GRIPPER_LINK2A/2B branches with scaled meshes and revolute joints in QARM.urdf - wire gripper-link2A/2B meshes into Panda viewer fallback map so they render with the new URDF links

File: sim/qarm/urdf/QARM.urdf (robot description, URDF)
Before this commit: robot QARM, 8 links, 7 joints
Links:
- added link GRIPPER_LINK1B, mass 0.02; collision mesh filename=package://QARM/meshes/gripper-link1b.stl scale=0.001 0.001 0.001; visual mesh filename=package://QARM/meshes/gripper-link1b.stl scale=0.001 0.001 0.001
- added link GRIPPER_LINK2A, mass 0.02; collision mesh filename=package://QARM/meshes/gripper-link2a.stl scale=0.001 0.001 0.001; visual mesh filename=package://QARM/meshes/gripper-link2a.stl scale=0.001 0.001 0.001
- added link GRIPPER_LINK2B, mass 0.02; collision mesh filename=package://QARM/meshes/gripper-link2b.stl scale=0.001 0.001 0.001; visual mesh filename=package://QARM/meshes/gripper-link2b.stl scale=0.001 0.001 0.001
Joints:
- added joint GRIPPER_JOINT1B: type revolute, parent GRIPPER_LINK1A, child GRIPPER_LINK1B, origin xyz=-0.003 -0.0347 0.0604 rpy=0 0 0, axis 1 0 0, limit lower=-3.14159 upper=3.14159 effort=0 velocity=0
- added joint GRIPPER_JOINT2A: type revolute, parent GRIPPER_BASE, child GRIPPER_LINK2A, origin xyz=0.02 0.0303 0.0406 rpy=0 0 0, axis 1 0 0, limit lower=-3.14159 upper=3.14159 effort=0 velocity=0
- added joint GRIPPER_JOINT2B: type revolute, parent GRIPPER_LINK2A, child GRIPPER_LINK2B, origin xyz=-0.003 0.0347 0.0604 rpy=0 0 0, axis 1 0 0, limit lower=-3.14159 upper=3.14159 effort=0 velocity=0
